Commit message: feat: adding ik piper

File: assets/piper/piper.urdf (robot description, URDF)
Before this commit: robot dual_piper_description, 19 links, 18 joints
Joints:
- joint der_joint1: axis 0 0 1 -> 0 0 -1; limit lower=-2.618 upper=2.168 effort=20000 velocity=3.14 -> lower=-2.168 upper=2.618 effort=20000 velocity=3.14
- joint der_joint2: axis 0 0 1 -> 0 0 -1; limit lower=0 upper=3.14 effort=20000 velocity=3.14 -> lower=-3.14 upper=0 effort=20000 velocity=3.14
- joint der_joint3: axis 0 0 1 -> 0 0 -1; limit lower=-2.967 upper=0 effort=1000 velocity=3.14 -> lower=0 upper=2.967 effort=1000 velocity=3.14
- joint der_joint4: axis 0 0 1 -> 0 0 -1
- joint der_joint5: axis 0 0 1 -> 0 0 -1
- joint der_joint6: axis 0 0 1 -> 0 0 -1
