Commit message: feat: solver v0.1

File: assets/piper/piper.urdf (robot description, URDF)
Before this commit: robot dual_piper, 23 links, 22 joints
Links:
- added link left_tcp
- added link right_tcp
- link left_base_link: geometry collision mesh filename=package://piper_description/meshes/base_link.STL; visual mesh filename=package://piper_description/meshes/base_link.STL
- link left_gripper_base: geometry collision mesh filename=package://piper_description/meshes/gripper_base.STL; visual mesh filename=package://piper_description/meshes/gripper_base.STL
- link left_link1: geometry collision mesh filename=package://piper_description/meshes/link1.STL; visual mesh filename=package://piper_description/meshes/link1.STL
- link left_link2: geometry collision mesh filename=package://piper_description/meshes/link2.STL; visual mesh filename=package://piper_description/meshes/link2.STL
- link left_link3: geometry collision mesh filename=package://piper_description/meshes/link3.STL; visual mesh filename=package://piper_description/meshes/link3.STL
- link left_link4: geometry collision mesh filename=package://piper_description/meshes/link4.STL; visual mesh filename=package://piper_description/meshes/link4.STL
- link left_link5: geometry collision mesh filename=package://piper_description/meshes/link5.STL; visual mesh filename=package://piper_description/meshes/link5.STL
- link left_link6: geometry collision mesh filename=package://piper_description/meshes/link6.STL; visual mesh filename=package://piper_description/meshes/link6.STL
- link left_link7: geometry collision mesh filename=package://piper_description/meshes/link7.STL; visual mesh filename=package://piper_description/meshes/link7.STL
- link left_link8: geometry collision mesh filename=package://piper_description/meshes/link8.STL; visual mesh filename=package://piper_description/meshes/link8.STL
- link right_base_link: geometry collision mesh filename=package://piper_description/meshes/base_link.STL; visual mesh filename=package://piper_description/meshes/base_link.STL
- link right_gripper_base: geometry collision mesh filename=package://piper_description/meshes/gripper_base.STL; visual mesh filename=package://piper_description/meshes/gripper_base.STL
- link right_link1: geometry collision mesh filename=package://piper_description/meshes/link1.STL; visual mesh filename=package://piper_description/meshes/link1.STL
- link right_link2: geometry collision mesh filename=package://piper_description/meshes/link2.STL; visual mesh filename=package://piper_description/meshes/link2.STL
- link right_link3: geometry collision mesh filename=package://piper_description/meshes/link3.STL; visual mesh filename=package://piper_description/meshes/link3.STL
- link right_link4: geometry collision mesh filename=package://piper_description/meshes/link4.STL; visual mesh filename=package://piper_description/meshes/link4.STL
- link right_link5: geometry collision mesh filename=package://piper_description/meshes/link5.STL; visual mesh filename=package://piper_description/meshes/link5.STL
- link right_link6: geometry collision mesh filename=package://piper_description/meshes/link6.STL; visual mesh filename=package://piper_description/meshes/link6.STL
- link right_link7: geometry collision mesh filename=package://piper_description/meshes/link7.STL; visual mesh filename=package://piper_description/meshes/link7.STL
- link right_link8: geometry collision mesh filename=package://piper_description/meshes/link8.STL; visual mesh filename=package://piper_description/meshes/link8.STL
Joints:
- added joint left_link6_to_tcp: type fixed, parent left_link6, child left_tcp, origin xyz=0 0 0.145 rpy=0 0 0
- added joint right_link6_to_tcp: type fixed, parent right_link6, child right_tcp, origin xyz=0 0 0.145 rpy=0 0 0
- joint world_to_left: origin xyz=0.0 0.3 0.0 rpy=0 0 0 -> xyz=0.0 0.35 0.0 rpy=0 0 0
- joint world_to_right: origin xyz=0.0 -0.3 0.0 rpy=0 0 0 -> xyz=0.0 -0.35 0.0 rpy=0 0 0

Commit message: fix(piper): expose one gripper joint per arm
What changed:
- Treat Piper joint8 as a mimic/equality-coupled finger while keeping its visual and collision geometry.
- Configure Piper runtime as six arm joints plus joint7 gripper per side with a 14-value home_q.
- Add registry coverage for the 14-DOF Piper layout and update teleop home indices.

Verification:
- uv run pytest tests/robots/test_registry.py tests/scripts/test_teleop_sim.py tests/scripts/test_conversion_gripper.py -q — passed

File: assets/piper/piper.urdf (robot description, URDF)
Before this commit: robot dual_piper, 25 links, 24 joints
Joints:
- joint left_joint8: mimic (none) -> joint=left_joint7 multiplier=-1 offset=0
- joint right_joint8: mimic (none) -> joint=right_joint7 multiplier=-1 offset=0
