Commit message: fix(openarm): prevent closed gripper overlap
What changed:
- Offset both simulated finger pairs to preserve clearance at the closed 0 mm position.
- Add a regression test for the URDF finger origins while retaining real-backend gripper semantics.

Verification:
- JAX_PLATFORMS=cpu uv run pytest -q tests/robots/test_registry.py -k 'openarm_closed_fingers or openarm_gripper_mapping' — 2 passed

File: assets/openarm/urdf/openarm_v1.urdf (robot description, URDF)
Before this commit: robot openarm, 24 links, 23 joints
Joints:
- joint openarm_left_finger_joint1: origin xyz=0.0 0.0 0.1025 rpy=0 0 0 -> xyz=0.0 -0.008 0.1025 rpy=0 0 0
- joint openarm_left_finger_joint2: origin xyz=0.0 -0.0 0.1025 rpy=0 0 0 -> xyz=0.0 0.008 0.1025 rpy=0 0 0
- joint openarm_right_finger_joint1: origin xyz=0.0 0.0 0.1025 rpy=0 0 0 -> xyz=0.0 -0.008 0.1025 rpy=0 0 0
- joint openarm_right_finger_joint2: origin xyz=0.0 -0.0 0.1025 rpy=0 0 0 -> xyz=0.0 0.008 0.1025 rpy=0 0 0
