Commit message: fix(yam): preserve jaw aperture and motor finish
- Correct the official linear gripper convention and preserve demonstrated aperture in meters during YAM replay.\n- Split upstream link visuals into white structure and black motor housings without changing kinematics.

File: assets/yam/yam_bimanual.urdf (robot description, URDF)
Before this commit: robot yam_bimanual, 23 links, 22 joints
Links:
- link left_link2: geometry visual mesh filename=meshes/arm/link2_arm.stl; visual mesh filename=meshes/arm/link2_elbow.stl
- link left_link3: geometry visual mesh filename=meshes/arm/link3_arm.stl; visual mesh filename=meshes/arm/link3_elbow.stl
- link right_link2: geometry visual mesh filename=meshes/arm/link2_arm.stl; visual mesh filename=meshes/arm/link2_elbow.stl
- link right_link3: geometry visual mesh filename=meshes/arm/link3_arm.stl; visual mesh filename=meshes/arm/link3_elbow.stl
